File: OSDMG0v1/opemGBZ.brd (EAGLE design)
At the start: 81.3 x 69.4 mm, 44 parts, among them IC1 TP4056, J1 SJ2-35954D-SMT-TR, U1 FS8205, U2 FS312F-G, U3 MT3608

Commit message: update Eagle
Parts:
- added SW0, SW1: (no value), wirepad:SMD1,27-2,54
Connections:
- new net L-OUT1: SW0.1
- net BAT+: now also SW1.1
Changed lines of the file:
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@@
 <attribute name="PRODUCT_TYPE" value="Connector" x="31.089596875" y="1.828796875" size="1.778" layer="27" display="off"/>
 </element>
+<element name="SW0" library="wirepad" library_urn="urn:adsk.eagle:library:412" package="SMD1,27-2,54" package3d_urn="urn:adsk.eagle:package:30839/1" value="" x="-107.47248125" y="-67.54368125"/>
+<element name="SW1" library="wirepad" library_urn="urn:adsk.eagle:library:412" package="SMD1,27-2,54" package3d_urn="urn:adsk.eagle:package:30839/1" value="" x="-111.13008125" y="-67.84848125"/>
 </elements>
 <signals>
@@
 <contactref element="R6" pad="2"/>
 <contactref element="C1" pad="1"/>
-<contactref element="U3" pad="5"/>
 <contactref element="U3" pad="4"/>
 <contactref element="L1" pad="2"/>
+<contactref element="U3" pad="5"/>
+<contactref element="SW1" pad="1"/>
+<wire x1="-68.3006" y1="1.27" x2="-111.13008125" y2="-67.84848125" width="0" layer="19" extent="1-1"/>
 <wire x1="-62.23" y1="3.94" x2="-68.3006" y2="1.27" width="0" layer="19" extent="1-1"/>
 <wire x1="-61.28" y1="3.94" x2="-62.23" y2="3.94" width="0" layer="19" extent="1-1"/>
@@
 <wire x1="-81.442559375" y1="-22.920959375" x2="-81.3816" y2="-61.2648" width="0" layer="19" extent="1-1"/>
 </signal>
+<signal name="L-OUT1">
+<contactref element="SW0" pad="1"/>
+</signal>
 </signals>

Commit message: update
Connections:
- new net N$30: C4.2, R6.1, U2.5
- net GND: no longer C4.2, R6.1, U2.5
Changed lines of the file:
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@@
 <contactref element="C3" pad="2"/>
 <contactref element="R5" pad="1"/>
-<contactref element="R6" pad="1"/>
 <contactref element="R7" pad="1"/>
-<contactref element="C4" pad="2"/>
 <contactref element="C1" pad="2"/>
 <contactref element="R3" pad="1"/>
 <contactref element="C2" pad="2"/>
 <contactref element="U1" pad="3"/>
-<contactref element="U2" pad="5"/>
 <contactref element="U3" pad="2"/>
 <contactref element="JP4" pad="2"/>
@@
 <contactref element="USBC" pad="A1"/>
 <contactref element="USBC" pad="B1"/>
-<wire x1="28.339596875" y1="6.458796875" x2="28.089596875" y2="5.258796875" width="0" layer="19" extent="1-1"/>
-<wire x1="-111.8616" y1="-61.2648" x2="28.339596875" y2="6.458796875" width="0" layer="19" extent="1-1"/>
-<wire x1="33.839596875" y1="6.458796875" x2="28.339596875" y2="6.458796875" width="0" layer="19" extent="1-1"/>
-<wire x1="34.089596875" y1="5.258796875" x2="33.839596875" y2="6.458796875" width="0" layer="19" extent="1-1"/>
-<wire x1="-72.39" y1="-24.13" x2="33.839596875" y2="6.458796875" width="0" layer="19" extent="1-1"/>
+<wire x1="-72.39" y1="-24.13" x2="-111.8616" y2="-61.2648" width="0" layer="19" extent="1-1"/>
 <wire x1="-62.23" y1="1.14" x2="-72.39" y2="-24.13" width="0" layer="19" extent="1-1"/>
-<wire x1="-58.42" y1="3.94" x2="-62.23" y2="1.14" width="0" layer="19" extent="1-1"/>
-<wire x1="-53.66" y1="1.14" x2="-58.42" y2="3.94" width="0" layer="19" extent="1-1"/>
-<wire x1="-51.01" y1="23.495" x2="-58.42" y2="3.94" width="0" layer="19" extent="1-1"/>
+<wire x1="-53.66" y1="1.14" x2="-62.23" y2="1.14" width="0" layer="19" extent="1-1"/>
+<wire x1="-51.01" y1="23.495" x2="-53.66" y2="1.14" width="0" layer="19" extent="1-1"/>
 <wire x1="-51.01" y1="26.035" x2="-51.01" y2="23.495" width="0" layer="19" extent="1-1"/>
 <wire x1="-38.69" y1="25.4" x2="-51.01" y2="26.035" width="0" layer="19" extent="1-1"/>
 <wire x1="-47.41" y1="41.91" x2="-51.01" y2="26.035" width="0" layer="19" extent="1-1"/>
-<wire x1="-49.95" y1="45.72" x2="-47.41" y2="41.91" width="0" layer="19" extent="1-1"/>
 <wire x1="-32.6" y1="46.99" x2="-47.41" y2="41.91" width="0" layer="19" extent="1-1"/>
 <wire x1="-28.79" y1="46.99" x2="-32.6" y2="46.99" width="0" layer="19" extent="1-1"/>
 <wire x1="-19.9" y1="50.8" x2="-28.79" y2="46.99" width="0" layer="19" extent="1-1"/>
-<wire x1="-17.36" y1="46.99" x2="-19.9" y2="50.8" width="0" layer="19" extent="1-1"/>
-<wire x1="-14.56" y1="34.29" x2="-17.36" y2="46.99" width="0" layer="19" extent="1-1"/>
+<wire x1="-14.56" y1="34.29" x2="-19.9" y2="50.8" width="0" layer="19" extent="1-1"/>
 <wire x1="7.18311875" y1="42.0217625" x2="-14.56" y2="34.29" width="0" layer="19" extent="1-1"/>
 <wire x1="16.256" y1="32.8168" x2="7.18311875" y2="42.0217625" width="0" layer="19" extent="1-1"/>
@@
 <wire x1="67.828159375" y1="61.569596875" x2="74.5744" y2="46.8376" width="0" layer="19" extent="1-1"/>
 <wire x1="53.329840625" y1="54.620159375" x2="67.828159375" y2="61.569596875" width="0" layer="19" extent="1-1"/>
+<wire x1="33.839596875" y1="6.458796875" x2="33.37405625" y2="26.551034375" width="0" layer="19" extent="1-1"/>
+<wire x1="34.089596875" y1="5.258796875" x2="33.839596875" y2="6.458796875" width="0" layer="19" extent="1-1"/>
+<wire x1="28.339596875" y1="6.458796875" x2="33.839596875" y2="6.458796875" width="0" layer="19" extent="1-1"/>
+<wire x1="28.089596875" y1="5.258796875" x2="28.339596875" y2="6.458796875" width="0" layer="19" extent="1-1"/>
 </signal>
 <signal name="N$9">
@@
 <contactref element="SW0" pad="1"/>
 </signal>
+<signal name="N$30">
+<contactref element="C4" pad="2"/>
+<contactref element="U2" pad="5"/>
+<contactref element="R6" pad="1"/>
+<wire x1="-49.95" y1="45.72" x2="-58.42" y2="3.94" width="0" layer="19" extent="1-1"/>
+<wire x1="-17.36" y1="46.99" x2="-49.95" y2="45.72" width="0" layer="19" extent="1-1"/>
+</signal>
 </signals>

Commit message: Eagle finished
Parts:
- removed SW0: (no value), wirepad:SMD1,27-2,54
- added SW2: (no value), wirepad:SMD1,27-2,54
- moved SW1 211.9 mm to (75.3, 32.7), flipped to the bottom
- moved JP2 178.6 mm to (31.3, 63.4)
- moved SPK- 174.2 mm to (52.2, 5.97), flipped to the bottom, turned to 90 degrees
- moved SPK+ 172.9 mm to (52.2, 9.39), flipped to the bottom, turned to 90 degrees
- moved JP4 159.1 mm to (56.6, 67.3)
- moved L1 150.0 mm to (73.1, 42.7), flipped to the bottom
- moved JP3 145.3 mm to (62.3, 33.5), turned to 180 degrees
- moved U$1 136.4 mm to (18.5, 47.2), flipped to the bottom
- moved GND 115.3 mm to (5.55, 39.0), flipped to the bottom, turned to 90 degrees
- moved R-IN 114.3 mm to (5.55, 42.4), flipped to the bottom, turned to 90 degrees
- moved L-IN 113.6 mm to (5.55, 45.8), flipped to the bottom, turned to 90 degrees
- moved R-OUT 113.0 mm to (5.55, 49.3), flipped to the bottom, turned to 90 degrees
- moved L-OUT 112.7 mm to (5.55, 52.7), flipped to the bottom, turned to 90 degrees
- moved D1 110.4 mm to (45.2, 29.4), flipped to the bottom
- moved U3 107.8 mm to (44.7, 15.9), flipped to the bottom, turned to 90 degrees
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Connections:
- removed net L-OUT1: SW0.1
- new net N$31: C1.1, L1.2, SW2.1, U3.4, U3.5
- net BAT+: now also JP3.1; no longer C1.1, L1.2, U3.4, U3.5
- net BAT-: now also JP3.2, U1.6; no longer U1.1
- net GND: now also U1.4; no longer U1.3
- net N$16: now also U1.3; no longer U1.4
- net N$17: now also U1.1; no longer U1.6
Routing:
- net 5V: track 0.00 -> 89.7 mm
- net N$22: track 0.00 -> 83.9 mm
- net N$28: track 0.00 -> 77.0 mm, vias 0 -> 4
- net N$29: track 0.00 -> 75.2 mm, vias 0 -> 2
- net BAT+: track 0.00 -> 71.6 mm, vias 0 -> 2
- net N$25: track 0.00 -> 65.7 mm, vias 0 -> 2
- net N$31: track 0.00 -> 59.7 mm
- net N$19: track 0.00 -> 59.6 mm, vias 0 -> 3
- net N$26: track 0.00 -> 58.8 mm, vias 0 -> 2
- net N$9: track 0.00 -> 58.3 mm
- net N$6: track 0.00 -> 50.4 mm, vias 0 -> 2
- net N$8: track 0.00 -> 47.9 mm
- net VBUS: track 0.00 -> 47.5 mm
- net N$5: track 0.00 -> 47.4 mm, vias 0 -> 2
- net R-OUT: track 0.00 -> 47.1 mm
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- added copper zone on layer 1, net GND
- added copper zone on layer 16, net GND
Other:
- board text removed: "+"
