File: OSDMG0v2/openGBZv2.brd (EAGLE design)
At the start: 81.3 x 69.4 mm, 80 parts, among them IC1 ATMEGA32U4-AU, IC2 TP4056, J1 SJ2-35954D-SMT-TR, T1 BC846S, U1 FS8205, U3 FS312F-G, X3 16MHz

Commit message: update and finish all projects
Parts:
- moved C4 0.25 mm to (51.3, 50.7)
Routing:
- net GND: track 2.61 -> 76.5 mm, vias 0 -> 27
- net BAT+: track 115.4 -> 110.7 mm
- net N$35: track 35.3 -> 38.9 mm
- net D-: track 93.1 -> 94.8 mm
- net D9/A10: track 51.7 -> 52.8 mm
- net 5V: track 205.5 -> 206.1 mm
- added copper zone on layer 1, net GND
- added copper zone on layer 16, net GND
Other:
- board text added: "Audio"
- board text added: "BNT R/L"
- board text added: "L"
- board text added: "R"
